File: KiCad/TapBadge/TapBadge.sch (KiCad schematic (older format))
At the start: 30 parts

Commit message: Completed rev1 PCB
Parts:
- removed D?: LED_RABG, LED_SMD:LED_Avago_PLCC4_3.2x2.8mm_CW, symbol Device:LED_RABG
- added D2: WS2812B, LED_SMD:LED_SK6812MINI_PLCC4_3.5x3.5mm_P1.75mm, symbol LED:WS2812B
- added SW1, SW2: SW_Push, Button_Switch_SMD:SW_SPST_B3U-1000P, symbol Switch:SW_Push
- AE1: renamed from AE?; footprint (none) -> RF_Antenna:Texas_SWRA117D_2.4GHz_Left; LCSC (none) -> Ignore
- C1, C3: renamed from C?; footprint (none) -> Capacitor_SMD:C_0603_1608Metric_Pad1.05x0.95mm_HandSolder; LCSC (none) -> C87152
- C2, C4, C5: renamed from C?; footprint (none) -> Capacitor_SMD:C_0603_1608Metric_Pad1.05x0.95mm_HandSolder; LCSC (none) -> C1597
- D1: renamed from D?; LCSC (none) -> Ignore
- D3: renamed from D?; footprint (none) -> Diode_SMD:D_0603_1608Metric_Pad1.05x0.95mm_HandSolder; LCSC (none) -> C189957
- ESP1: renamed from ESP?; footprint (none) -> Package_DFN_QFN:QFN-48-1EP_7x7mm_P0.5mm_EP5.15x5.15mm; LCSC (none) -> C193707
- J1: renamed from J?; footprint (none) -> Connector_USB:USB_Micro-B_GCT_USB3076-30-A; LCSC (none) -> C132562
- J2: renamed from J?; footprint (none) -> TestPoint:TestPoint_THTPad_D1.5mm_Drill0.7mm; LCSC (none) -> Ignore
- M1: renamed from M?; footprint (none) -> Connector_PinHeader_2.00mm:PinHeader_1x02_P2.00mm_Vertical; LCSC (none) -> Ignore
- Q1, Q2, Q3, Q4: renamed from Q?; footprint (none) -> Package_TO_SOT_SMD:SOT-23; LCSC (none) -> C23869
- R1, R11, R2, R3, R5, R6, R7: renamed from R?; footprint (none) -> Resistor_SMD:R_0603_1608Metric_Pad1.05x0.95mm_HandSolder; LCSC (none) -> C25804
- R10, R9: renamed from R?; footprint (none) -> Resistor_SMD:R_0603_1608Metric_Pad1.05x0.95mm_HandSolder; LCSC (none) -> C25803
- R4, R8: renamed from R?; footprint (none) -> Resistor_SMD:R_0603_1608Metric_Pad1.05x0.95mm_HandSolder; LCSC (none) -> C4190
- U1: renamed from U?; LCSC (none) -> C80225
- U2: renamed from U?; LCSC (none) -> Ignore
Connections:
- net labels added: RGB_IO
- net labels removed: CH_STAT, RGB_B, RGB_G, RGB_R
- wire segments 107 -> 108

Commit message: Once used KiCAD 5 >.>
Parts:
- ESP1: symbol esp32pico_d4:ESP32PICO_D4 -> TapBadge-rescue:ESP32PICO_D4-esp32pico_d4
Changed lines of the file:
@@
 $EndDescr
 $Comp
-L esp32pico_d4:ESP32PICO_D4 ESP1
+L TapBadge-rescue:ESP32PICO_D4-esp32pico_d4 ESP1
 U 1 1 5B93C22A
 P 6225 4675
